File: avionics/Gables G3021 Audio Control Panel and Headphone Jack/schematics/OASIS_Card_v1/OASIS_Card.kicad_pcb (KiCad board)
At the start: 2 copper layers, 49 parts, among them U1 CD4051B, U3 LTC1044

Commit message: OASIS schematics
Parts:
- moved U3 63.1 mm to (129.8, 128.3)
- moved C12 63.1 mm to (133.0, 123.5)
- moved C13 63.1 mm to (126.3, 117.5)
- moved R11 12.3 mm to (114.7, 87.6)
- moved R12 12.3 mm to (114.7, 90.2)
- moved R13 12.3 mm to (114.7, 92.7)
- moved R14 12.3 mm to (114.7, 95.2)
- moved R15 12.3 mm to (114.7, 97.8)
- moved R16 12.3 mm to (114.7, 100.3)
- moved R17 12.3 mm to (114.7, 102.9)
- moved R18 12.3 mm to (114.7, 105.4)
- moved C1 12.3 mm to (122.6, 87.6)
- moved C2 12.3 mm to (122.6, 90.2)
- moved C3 12.3 mm to (122.6, 92.7)
- moved C4 12.3 mm to (122.6, 95.2)
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- renumbered C5 to C2, C2 to C3, C6 to C4, C3 to C5, C7 to C6, C4 to C7, D4 to D1, D3 to D2, D2 to D3, D1 to D4, R9 to R11, R10 to R12, R11 to R13, R12 to R14, R13 to R15, R14 to R16, R15 to R17, R16 to R18, R20 to R21, R19 to R22, R18 to R23, R17 to R24
Routing:
- net Net-(A2-D11): track 0.00 -> 88.2 mm
- net Net-(A2-D10): track 0.00 -> 87.7 mm
- net Net-(A2-D12): track 0.00 -> 85.1 mm
- net +5V: track 0.00 -> 76.3 mm, vias 0 -> 1
- net Net-(A2-D13): track 0.00 -> 21.5 mm
- net Net-(U1-X6): track 0.00 -> 11.0 mm
- net Net-(U1-X7): track 0.00 -> 9.97 mm
- net Net-(U1-X5): track 0.00 -> 9.55 mm, vias 0 -> 1
- net Net-(A2-D9): track 0.00 -> 5.76 mm
- net Net-(A2-D8): track 0.00 -> 5.76 mm
- net Net-(A2-D7): track 0.00 -> 5.76 mm
- net Net-(A2-D6): track 0.00 -> 5.76 mm
- net Net-(A2-D5): track 0.00 -> 5.76 mm
- net Net-(A2-D4): track 0.00 -> 5.76 mm
- net Net-(A2-D3): track 0.00 -> 5.76 mm
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
Commit message: audio boss
Parts:
- moved H3 82.0 mm to (95.5, 112.5)
- moved H1 82.0 mm to (95.5, 96.6)
- moved H2 82.0 mm to (95.5, 104.6)
- moved H5 82.0 mm to (95.5, 120.5)
- moved U3 73.1 mm to (198.9, 104.4)
- moved C11 73.1 mm to (183.7, 106.2)
- moved C10 73.1 mm to (183.7, 103.4)
- moved C12 73.1 mm to (202.1, 99.6)
- moved C13 73.1 mm to (195.4, 93.6)
- moved TP1 68.9 mm to (84.1, 95.7), turned to 90 degrees
- moved TP4 61.3 mm to (83.3, 113.2), turned to 90 degrees
- moved TP2 61.0 mm to (83.6, 100.0), turned to 90 degrees
- moved TP3 58.3 mm to (83.3, 104.6), turned to 90 degrees
- moved TP6 50.7 mm to (83.6, 108.9)
- moved U1 19.2 mm to (139.7, 111.3), turned to 180 degrees
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Routing:
- net Net-(A2-D11): track 88.2 -> 4.68 mm
- net Net-(A2-D10): track 87.7 -> 4.70 mm
- net Net-(A2-D12): track 85.1 -> 4.70 mm
- net Net-(U1-X0): track 35.1 -> 4.57 mm
- net Net-(U1-X1): track 31.2 -> 4.57 mm
- net Net-(U1-X2): track 27.5 -> 4.57 mm
- net Net-(U1-X7): track 9.97 -> 26.4 mm
- net Net-(U1-X5): track 9.55 -> 22.3 mm, vias 1 -> 0
- net Net-(U1-X3): track 26.9 -> 19.5 mm
- net Net-(U1-X6): track 11.0 -> 16.4 mm
- net +5V: track 76.3 -> 80.3 mm
- net Net-(U1-X4): track 9.97 -> 13.2 mm, vias 0 -> 1

Commit message: OASIS card layout
Parts:
- added J1: Conn_02x08_Top_Bottom, Jurassic_Jets_Footprints:2x08_3.5mm_Phoenix_Connector_knockoff, F.Cu at (116.3, 101.9)
- added J3: 12v DC, TerminalBlock_Phoenix:TerminalBlock_Phoenix_MKDS-1,5-2-5.08_1x02_P5.08mm_Horizontal, F.Cu at (171.6, 126.2)
- added J4: AudioJack3_Ground_Switch, Jurassic_Jets_Footprints:TRS_2_Pole_THT, F.Cu at (204.9, 100.2)
- added J7: Piggyback Master, Connector_PinHeader_2.54mm:PinHeader_1x05_P2.54mm_Vertical, B.Cu at (181.9, 87.6)
- added J8: Piggyback Slave, Connector_PinHeader_2.54mm:PinHeader_1x05_P2.54mm_Vertical, B.Cu at (181.9, 129.3)
- added J9: 12v DC, TerminalBlock_Phoenix:TerminalBlock_Phoenix_MKDS-1,5-2-5.08_1x02_P5.08mm_Horizontal, F.Cu at (108.5, 90.2)
- TP2, TP3, TP4: footprint Connector_Pin:Pin_D0.9mm_L10.0mm_W2.4mm_FlatFork -> Connector_PinHeader_2.54mm:PinHeader_1x01_P2.54mm_Vertical
- moved TP6 106.4 mm to (188.7, 93.0)
- moved H2 105.0 mm to (198.1, 127.0)
- moved H1 102.8 mm to (198.1, 90.4)
- moved TP2 92.9 mm to (175.0, 116.3), turned to -90 degrees
- moved TP4 92.0 mm to (175.0, 105.2), turned to -90 degrees
- moved TP3 91.9 mm to (175.0, 110.7), turned to -90 degrees
- moved C11 68.0 mm to (117.3, 91.2)
- moved C10 68.0 mm to (117.4, 88.4)
- moved TP1 56.5 mm to (130.6, 127.8)
- moved H3 36.6 mm to (124.5, 90.2)
- moved H5 29.6 mm to (124.5, 126.7)
- moved U3 21.2 mm to (178.2, 100.1)
- moved C12 21.2 mm to (181.3, 95.3)
- moved C13 21.2 mm to (174.7, 89.3)
- moved C9 10.9 mm to (129.5, 96.7), turned to 90 degrees
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Connections:
- TP1 pad 2: GND -> unconnected-(TP1-Pad2)
Routing:
- net +12V: track 0.00 -> 207.7 mm, vias 0 -> 2
- net +5V: track 80.3 -> 207.7 mm, vias 1 -> 3
- net Net-(J8-Pin_1): track 0.00 -> 112.9 mm
- net -5V: track 5.26 -> 101.4 mm
- net Net-(A2-D12): track 4.70 -> 71.5 mm
- net Net-(A2-D11): track 4.68 -> 69.3 mm
- net Net-(A2-D10): track 4.70 -> 66.0 mm
- net Net-(A2-D2): track 5.76 -> 60.8 mm
- net Net-(A2-D3): track 5.76 -> 58.8 mm
- net Net-(A2-D4): track 5.76 -> 56.9 mm
- net Net-(A2-D5): track 5.76 -> 54.9 mm
- net Net-(A2-D6): track 5.76 -> 51.5 mm
- net Net-(A2-D7): track 5.76 -> 50.6 mm
- net Net-(A2-D8): track 5.76 -> 50.6 mm
- net Net-(A2-D9): track 5.76 -> 49.7 mm
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- added copper zone on B.Cu, net GND
- added copper zone on F.Cu, net GND
Other:
- board outline added: 106.4 x 46.2 mm

Commit message: more OASIS card stuff
Parts:
- added G***: LOGO, LOGO, F.Cu at (184.7, 122.5)
- added G***: LOGO, LOGO, B.Cu at (156.6, 108.5)
- TP2, TP3, TP4: footprint Connector_PinHeader_2.54mm:PinHeader_1x01_P2.54mm_Vertical -> TestPoint:TestPoint_Pad_2.5x2.5mm
- moved U3 9.31 mm to (169.9, 95.8), turned to 90 degrees
- moved C12 7.57 mm to (174.7, 98.9), turned to 180 degrees
- moved C13 7.52 mm to (180.3, 94.2), turned to 90 degrees
- moved C10 3.82 mm to (117.6, 92.2)
- moved C11 3.82 mm to (117.6, 95.0)
Routing:
- net +5V: track 207.7 -> 219.3 mm, vias 3 -> 4
- net GND: track 0.02 -> 10.7 mm, vias 10 -> 20
- net -5V: track 101.4 -> 108.7 mm, vias 0 -> 1
- net +12V: track 207.7 -> 202.2 mm, vias 2 -> 3
- net Net-(A2-D10): track 66.0 -> 69.0 mm
- net Net-(A2-D4): track 56.9 -> 59.7 mm
- net Net-(A2-D9): track 49.7 -> 52.5 mm
- net Net-(A2-D6): track 51.5 -> 53.1 mm
- net Net-(D3-K): track 5.01 -> 6.43 mm
- net Net-(A2-D12): track 71.5 -> 72.9 mm
- net Net-(D1-K): track 5.01 -> 6.43 mm
- net Net-(A2-D3): track 58.8 -> 60.2 mm
- net Net-(A2-D7): track 50.6 -> 52.0 mm
- net Net-(J8-Pin_1): track 112.9 -> 113.9 mm
- net Net-(A2-D11): track 69.3 -> 70.1 mm
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Other:
- board text added: "Jurassic Jets"
- board text added: "OASIS Mic Card v1"
- board text added: "{dblquote}uhhhh, radio check?{dblquote}"
