File: avionics/Gables G3021 Audio Control Panel and Headphone Jack/schematics/OASIS_Card_v1/OASIS_Card.kicad_sch (KiCad schematic)
At the start: 33 parts, among them J1 Mic Input, J2 Control Input, J3 12v DC IN, U1 CD4051B, U2 L7812

Commit message: OASIS schematic
Connections:
- net +5V: now also C9.1, U1.16 (VDD)
- net -5V: now reaches U1.7 (VEE)
Changed lines of the file:
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@@
+	(wire
+		(pts
+			(xy 160.02 102.87) (xy 154.94 102.87)
+		)
+		(stroke
+			(width 0)
+			(type default)
+		)
+	)
 	(wire
 		(pts
@@
 	(wire
 		(pts
+			(xy 160.02 101.6) (xy 160.02 102.87)
+		)
+		(stroke
+			(width 0)
+			(type default)
+		)
+	)
+	(wire
+		(pts
 			(xy 152.4 96.52) (xy 152.4 99.06)
 		)
@@
 		(pts
 			(xy 185.42 129.54) (xy 53.34 129.54)
+		)
+		(stroke
+			(width 0)
+			(type default)
+		)
+	)
+	(wire
+		(pts
+			(xy 154.94 102.87) (xy 154.94 96.52)
 		)
 		(stroke
@@
 	)
 	(symbol
+		(lib_id "power:-5V")
+		(at 160.02 101.6 0)
+		(unit 1)
+		(exclude_from_sim no)
+		(in_bom yes)
+		(on_board yes)
+		(dnp no)
+		(fields_autoplaced yes)
+		(property "Reference" "#PWR011"
+			(at 160.02 105.41 0)
+			(effects
+				(font
+					(size 1.27 1.27)
+				)
+				(hide yes)
+			)
+		)
+		(property "Value" "-5V"
+			(at 160.02 96.52 0)
+			(effects
+				(font
+					(size 1.27 1.27)
+				)
+			)
+		)
+		(property "Footprint" ""
+			(at 160.02 101.6 0)
+			(effects
+				(font
+					(size 1.27 1.27)
+				)
+				(hide yes)
+			)
+		)
+		(property "Datasheet" ""
+			(at 160.02 101.6 0)
+			(effects
+				(font
+					(size 1.27 1.27)
+				)
+				(hide yes)
+			)
+		)
+		(property "Description" "Power symbol creates a global label with name \"-5V\""
+			(at 160.02 101.6 0)
+			(effects
+				(font
+					(size 1.27 1.27)
+				)
+				(hide yes)
+			)
+		)
+		(pin "1"
+		)
+		(instances
+			(project ""
+				(path "/6941f5ac-693b-4b10-8fb5-654c90b13202"
+					(reference "#PWR011")
+					(unit 1)
+				)
+			)
+		)
+	)
+	(symbol
 		(lib_id "Connector:Screw_Terminal_01x08")
 		(at 21.59 81.28 0)
@@
 					(unit 1)
 				)
+			)
+		)
+	)
+	(symbol
+		(lib_id "power:+5V")
+		(at 149.86 48.26 0)
+		(unit 1)
+		(exclude_from_sim no)
+		(in_bom yes)
+		(on_board yes)
+		(dnp no)
+		(fields_autoplaced yes)
+		(property "Reference" "#PWR010"
+			(at 149.86 52.07 0)
+			(effects
+				(font
+					(size 1.27 1.27)
+				)
+				(hide yes)
+			)
+		)
+		(property "Value" "+5V"
+			(at 149.86 43.18 0)
+			(effects
+				(font
+					(size 1.27 1.27)
+				)
+			)
+		)
+		(property "Footprint" ""
+			(at 149.86 48.26 0)
+			(effects
+				(font
+					(size 1.27 1.27)
+				)
+				(hide yes)
+			)
+		)
+		(property "Datasheet" ""
+			(at 149.86 48.26 0)
+			(effects
+				(font
+					(size 1.27 1.27)
+				)
+				(hide yes)
+			)
+		)
+		(property "Description" "Power symbol creates a global label with name \"+5V\""
+			(at 149.86 48.26 0)
+			(effects
+				(font
+					(size 1.27 1.27)
+				)
+				(hide yes)
+			)
+		)
+		(pin "1"
+		)
+		(instances
+			(project "OASIS_Card"
+				(path "/6941f5ac-693b-4b10-8fb5-654c90b13202"
+					(reference "#PWR010")
+					(unit 1)
+				)

Commit message: OASIS schematics
Parts:
- removed U2: L7812, Package_TO_SOT_THT:TO-220-3_Vertical, symbol Regulator_Linear:L7812
- added C12: 10pF, Capacitor_SMD:C_1206_3216Metric_Pad1.33x1.80mm_HandSolder, symbol Device:C
- added C13: 10uF, Capacitor_SMD:C_1206_3216Metric_Pad1.33x1.80mm_HandSolder, symbol Device:C
- added D1, D2, D3, D4: LED, LED_SMD:LED_0805_2012Metric, symbol Device:LED
- added H1, H2, H3, H5: MountingHole_Pad, MountingHole:MountingHole_3.2mm_M3_Pad, symbol Mechanical:MountingHole_Pad
- added J4: AudioJack3, symbol Connector_Audio:AudioJack3
- added J5: Control Signals Out, symbol Connector:Screw_Terminal_01x04
- added J6: 12v DC OUT, symbol Connector:Screw_Terminal_01x02
- added R17, R18, R19, R20: R_LED, Resistor_SMD:R_0805_2012Metric_Pad1.20x1.40mm_HandSolder, symbol Device:R
- added TP1: GND, Connector_PinHeader_2.54mm:PinHeader_1x02_P2.54mm_Vertical, symbol Connector:TestPoint_2Pole
- added TP2: +12v, Connector_Pin:Pin_D0.9mm_L10.0mm_W2.4mm_FlatFork, symbol Connector:TestPoint
- added TP3: +5v, Connector_Pin:Pin_D0.9mm_L10.0mm_W2.4mm_FlatFork, symbol Connector:TestPoint
- added TP4: -5v, Connector_Pin:Pin_D0.9mm_L10.0mm_W2.4mm_FlatFork, symbol Connector:TestPoint
- added TP6: MIC OUT, Connector_PinHeader_2.54mm:PinHeader_1x02_P2.54mm_Vertical, symbol Connector:TestPoint_2Pole
- added U3: LTC1044, Package_DIP:DIP-8_W7.62mm, symbol Regulator_SwitchedCapacitor:LTC1044
- U1: footprint (none) -> Package_DIP:DIP-16_W7.62mm
Connections:
- net +12V: now also A2.30 (VIN), J6.2 (Pin_2), TP2.1
- net +5V: now also A2.27 (+5V), R1.2, R2.2, R3.2, R4.2, R5.2, R6.2, R7.2, R8.2, R17.1, TP3.1, U3.8 (V+); no longer A2.30 (VIN)
- net -5V: now also C13.2, TP4.1, U3.5 (VOUT)
- net GND: now also C13.1, H1.1, H2.1, H3.1, H5.1, J6.1 (Pin_1), R18.2, R19.2, R20.2, TP1.1, TP1.2, U3.3 (GND); no longer R1.2, R2.2, R3.2, R4.2, R5.2, R6.2, R7.2, R8.2
- net at A2.13 (D10): now also U1.11 (A), D2.2 (A), J5.1 (Pin_1)
- net at A2.14 (D11): now also U1.10 (B), D3.2 (A), J5.2 (Pin_2)
- net at A2.15 (D12): now also U1.9 (C), D4.2 (A), J5.3 (Pin_3)
- net at A2.16 (D13): now also D1.1 (K), J5.4 (Pin_4)
- net at U1.3 (X): now also TP6.1
- new net: D2.1 (K), R18.1
- new net: D4.1 (K), R20.1
- new net: C12.2, U3.2 (CAP+)
- new net: C12.1, U3.4 (CAP-)
- new net: D1.2 (A), R17.2
- new net: D3.1 (K), R19.1
Other:
- note added: "wire up audio jack add missing footprints"
- moved on the sheet: C10, C11, J1, J3, R10, R11, R12, R13, R14, R15, R16, R9

Commit message: OASIS schematics
Parts:
- renumbered C5 to C2, C2 to C3, C6 to C4, C3 to C5, C7 to C6, C4 to C7, D4 to D1, D3 to D2, D2 to D3, D1 to D4, R9 to R11, R10 to R12, R11 to R13, R12 to R14, R13 to R15, R14 to R16, R15 to R17, R16 to R18, R20 to R21, R19 to R22, R18 to R23, R17 to R24
Changed lines of the file:
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@@
 		(on_board yes)
 		(dnp no)
-		(property "Reference" "R18"
+		(property "Reference" "R23"
 			(at 193.04 63.5 90)
 			(effects
@@
 			(project "OASIS_Card"
 				(path "/6941f5ac-693b-4b10-8fb5-654c90b13202"
-					(reference "R18")
+					(reference "R23")
 					(unit 1)
 				)
@@
 		(on_board yes)
 		(dnp no)
-		(property "Reference" "D4"
+		(property "Reference" "D1"
 			(at 180.086 72.39 0)
 			(effects
@@
 			(project "OASIS_Card"
 				(path "/6941f5ac-693b-4b10-8fb5-654c90b13202"
-					(reference "D4")
+					(reference "D1")
 					(unit 1)
 				)
@@
 		(on_board yes)
 		(dnp no)
-		(property "Reference" "R17"
+		(property "Reference" "R24"
 			(at 152.4 147.32 90)
 			(effects
@@
 			(project "OASIS_Card"
 				(path "/6941f5ac-693b-4b10-8fb5-654c90b13202"
-					(reference "R17")
+					(reference "R24")
 					(unit 1)
 				)
@@
 		(on_board yes)
 		(dnp no)
-		(property "Reference" "C3"
+		(property "Reference" "C5"
 			(at 94.996 82.55 90)
 			(effects
@@
 			(project "OASIS_Old_ACP_Signal_Interfacing_and_Switching_Card"
 				(path "/6941f5ac-693b-4b10-8fb5-654c90b13202"
-					(reference "C3")
+					(reference "C5")
 					(unit 1)
 				)
@@
 		(on_board yes)
 		(dnp no)
-		(property "Reference" "D3"
+		(property "Reference" "D2"
 			(at 180.086 67.31 0)
 			(effects
@@
 			(project "OASIS_Card"
 				(path "/6941f5ac-693b-4b10-8fb5-654c90b13202"
-					(reference "D3")
+					(reference "D2")
 					(unit 1)
 				)
@@
 		(on_board yes)
 		(dnp no)
-		(property "Reference" "D2"
+		(property "Reference" "D3"
 			(at 180.086 62.23 0)
 			(effects
@@
 			(project "OASIS_Card"
 				(path "/6941f5ac-693b-4b10-8fb5-654c90b13202"
-					(reference "D2")
+					(reference "D3")
 					(unit 1)
 				)
@@
 		(on_board yes)
 		(dnp no)
-		(property "Reference" "R12"
+		(property "Reference" "R14"
 			(at 46.99 67.31 90)
 			(effects
@@
 			(project "OASIS_Old_ACP_Signal_Interfacing_and_Switching_Card"
 				(path "/6941f5ac-693b-4b10-8fb5-654c90b13202"
-					(reference "R12")
+					(reference "R14")
 					(unit 1)
 				)
@@
 		(on_board yes)
 		(dnp no)
-		(property "Reference" "R19"
+		(property "Reference" "R22"
 			(at 193.04 68.58 90)
 			(effects
@@
 			(project "OASIS_Card"
 				(path "/6941f5ac-693b-4b10-8fb5-654c90b13202"
-					(reference "R19")
+					(reference "R22")
 					(unit 1)
 				)
@@
 		(on_board yes)
 		(dnp no)
-		(property "Reference" "R14"
+		(property "Reference" "R16"
 			(at 57.15 67.31 90)
 			(effects
@@
 			(project "OASIS_Old_ACP_Signal_Interfacing_and_Switching_Card"
 				(path "/6941f5ac-693b-4b10-8fb5-654c90b13202"
-					(reference "R14")
+					(reference "R16")
 					(unit 1)
 				)
@@
 		(on_board yes)
 		(dnp no)
-		(property "Reference" "C5"
+		(property "Reference" "C2"
 			(at 94.996 74.93 90)
 			(effects
@@
 			(project "OASIS_Old_ACP_Signal_Interfacing_and_Switching_Card"
 				(path "/6941f5ac-693b-4b10-8fb5-654c90b13202"
-					(reference "C5")
+					(reference "C2")
 					(unit 1)
 				)
@@
 		(on_board yes)
 		(dnp no)
-		(property "Reference" "R13"
+		(property "Reference" "R15"
 			(at 52.07 67.31 90)
 			(effects
@@
 			(project "OASIS_Old_ACP_Signal_Interfacing_and_Switching_Card"
 				(path "/6941f5ac-693b-4b10-8fb5-654c90b13202"
-					(reference "R13")
+					(reference "R15")
 					(unit 1)
 				)
@@
 		(on_board yes)
 		(dnp no)
-		(property "Reference" "R20"
+		(property "Reference" "R21"
 			(at 193.04 73.66 90)
 			(effects
@@
 			(project "OASIS_Card"
 				(path "/6941f5ac-693b-4b10-8fb5-654c90b13202"
-					(reference "R20")
+					(reference "R21")
 					(unit 1)
 				)
@@
 		(on_board yes)
 		(dnp no)
-		(property "Reference" "R16"
+		(property "Reference" "R18"
 			(at 67.31 67.31 90)
 			(effects
@@
 			(project "OASIS_Old_ACP_Signal_Interfacing_and_Switching_Card"
 				(path "/6941f5ac-693b-4b10-8fb5-654c90b13202"
-					(reference "R16")
+					(reference "R18")
 					(unit 1)
 				)
@@
 		(on_board yes)
 		(dnp no)
-		(property "Reference" "D1"
-			(at 162.8775 140.97 0)
+		(property "Reference" "D4"
+			(at 162.814 142.24 0)
 			(effects
 				(font
@@
 		)
 		(property "Value" "LED"
-			(at 162.8775 143.51 0)
+			(at 162.814 144.78 0)
 			(effects
 				(font
@@
 			(project ""
 				(path "/6941f5ac-693b-4b10-8fb5-654c90b13202"
-					(reference "D1")
+					(reference "D4")
 					(unit 1)
 				)
@@
 		(on_board yes)
 		(dnp no)
-		(property "Reference" "R15"
+		(property "Reference" "R17"
 			(at 62.23 67.31 90)
 			(effects
@@
 			(project "OASIS_Old_ACP_Signal_Interfacing_and_Switching_Card"
 				(path "/6941f5ac-693b-4b10-8fb5-654c90b13202"
-					(reference "R15")
+					(reference "R17")
 					(unit 1)
 				)
@@
 		(on_board yes)
 		(dnp no)
-		(property "Reference" "R11"
+		(property "Reference" "R13"
 			(at 41.91 67.31 90)
 			(effects
@@
 			(project "OASIS_Old_ACP_Signal_Interfacing_and_Switching_Card"
 				(path "/6941f5ac-693b-4b10-8fb5-654c90b13202"
-					(reference "R11")
+					(reference "R13")
 					(unit 1)
 				)
@@
 		(on_board yes)
 		(dnp no)
-		(property "Reference" "R10"
+		(property "Reference" "R12"
 			(at 36.83 67.31 90)
 			(effects
@@
 			(project "OASIS_Old_ACP_Signal_Interfacing_and_Switching_Card"
 				(path "/6941f5ac-693b-4b10-8fb5-654c90b13202"
-					(reference "R10")
+					(reference "R12")
 					(unit 1)
 				)
@@
 		(on_board yes)
 		(dnp no)
-		(property "Reference" "C4"
+		(property "Reference" "C7"
 			(at 105.156 87.63 90)
 			(effects
@@
 			(project "OASIS_Old_ACP_Signal_Interfacing_and_Switching_Card"
 				(path "/6941f5ac-693b-4b10-8fb5-654c90b13202"
-					(reference "C4")
+					(reference "C7")
 					(unit 1)
 				)
@@
 		(on_board yes)
 		(dnp no)
-		(property "Reference" "C2"
+		(property "Reference" "C3"
 			(at 84.836 77.47 90)
 			(effects
@@
 			(project "OASIS_Old_ACP_Signal_Interfacing_and_Switching_Card"
 				(path "/6941f5ac-693b-4b10-8fb5-654c90b13202"
-					(reference "C2")
+					(reference "C3")
 					(unit 1)
 				)
@@
 		(on_board yes)
 		(dnp no)
-		(property "Reference" "C7"
+		(property "Reference" "C6"
 			(at 115.316 85.09 90)
 			(effects
@@
 			(project "OASIS_Old_ACP_Signal_Interfacing_and_Switching_Card"
 				(path "/6941f5ac-693b-4b10-8fb5-654c90b13202"
-					(reference "C7")
+					(reference "C6")
 					(unit 1)
 				)
@@
 		(on_board yes)
 		(dnp no)
-		(property "Reference" "R9"
+		(property "Reference" "R11"
 			(at 31.75 67.31 90)
 			(effects
@@
 			(project "OASIS_Old_ACP_Signal_Interfacing_and_Switching_Card"
 				(path "/6941f5ac-693b-4b10-8fb5-654c90b13202"
-					(reference "R9")
+					(reference "R11")
 					(unit 1)
 				)
@@
 		(on_board yes)
 		(dnp no)
-		(property "Reference" "C6"
+		(property "Reference" "C4"
 			(at 105.156 80.01 90)
 			(effects
@@
 			(project "OASIS_Old_ACP_Signal_Interfacing_and_Switching_Card"
 				(path "/6941f5ac-693b-4b10-8fb5-654c90b13202"
-					(reference "C6")
+					(reference "C4")
 					(unit 1)
 				)

Commit message: OASIS card layout
Parts:
- removed J1: Mic Input, symbol Connector:Screw_Terminal_01x08
- removed J2: Control Input, symbol Connector:Screw_Terminal_01x08
- removed J4: AudioJack3, symbol Connector_Audio:AudioJack3
- added J1: Conn_02x08_Top_Bottom, Jurassic_Jets_Footprints:2x08_3.5mm_Phoenix_Connector_knockoff, symbol Connector_Generic:Conn_02x08_Top_Bottom
- added J4: AudioJack3_Ground_Switch, Jurassic_Jets_Footprints:TRS_2_Pole_THT, symbol Connector_Audio:AudioJack3_Ground_Switch
- added J7: Piggyback Master, Connector_PinHeader_2.54mm:PinHeader_1x05_P2.54mm_Vertical, symbol Connector:Conn_01x05_Socket
- added J8: Piggyback Slave, Connector_PinHeader_2.54mm:PinHeader_1x05_P2.54mm_Vertical, symbol Connector:Conn_01x05_Pin
- added J9: 12v DC, TerminalBlock_Phoenix:TerminalBlock_Phoenix_MKDS-1,5-2-5.08_1x02_P5.08mm_Horizontal, symbol Connector:Screw_Terminal_01x02
- J3: value 12v DC IN -> 12v DC; footprint (none) -> TerminalBlock_Phoenix:TerminalBlock_Phoenix_MKDS-1,5-2-5.08_1x02_P5.08mm_Horizontal
- TP2, TP3, TP4: footprint Connector_Pin:Pin_D0.9mm_L10.0mm_W2.4mm_FlatFork -> Connector_PinHeader_2.54mm:PinHeader_1x01_P2.54mm_Vertical
Connections:
- net +12V: now also J7.5 (Pin_5), J8.5 (Pin_5), J9.2 (Pin_2)
- net +5V: now also J7.4 (Pin_4), J8.4 (Pin_4)
- net -5V: now also J7.3 (Pin_3), J8.3 (Pin_3)
- net GND: now also J4.S, J7.2 (Pin_2), J8.2 (Pin_2), J9.1 (Pin_1); no longer TP1.2
- net at A2.6 (D3), R2.1: now also J1.10 (Pin_10)
- net at C5.1, R15.2: now also J1.5 (Pin_5)
- net at C1.1, R11.2: now also J1.1 (Pin_1)
- net at C2.1, R12.2: now also J1.2 (Pin_2)
- net at C3.1, R13.2: now also J1.3 (Pin_3)
- net at C4.1, R14.2: now also J1.4 (Pin_4)
- net at C6.1, R16.2: now also J1.6 (Pin_6)
- net at C7.1, R17.2: now also J1.7 (Pin_7)
- net at C8.1, R18.2: now also J1.8 (Pin_8)
- net at A2.10 (D7), R6.1: now also J1.14 (Pin_14)
- net at A2.11 (D8), R7.1: now also J1.15 (Pin_15)
- net at A2.12 (D9), R8.1: now also J1.16 (Pin_16)
- net at A2.5 (D2), R1.1: now also J1.9 (Pin_9)
- net at A2.7 (D4), R3.1: now also J1.11 (Pin_11)
- net at A2.8 (D5), R4.1: now also J1.12 (Pin_12)
- net at A2.9 (D6), R5.1: now also J1.13 (Pin_13)
- net at TP6.1, U1.3 (X): now also J4.T, J8.1 (Pin_1)
- new net: J4.R, J7.1 (Pin_1)
Other:
- note removed: "wire up audio jack add missing footprints"
- moved on the sheet: R1, R2, R3, R4, R5, R6, R7, R8

Commit message: more OASIS card stuff
Parts:
- TP2, TP3, TP4: footprint Connector_PinHeader_2.54mm:PinHeader_1x01_P2.54mm_Vertical -> TestPoint:TestPoint_Pad_2.5x2.5mm
Other:
- moved on the sheet: J4, J7, J8
