File: PCBs/OASIS_Audio_Card_v1/OASIS_Audio_Card_v1.kicad_sch (KiCad schematic)
At the start: 9 parts, among them J1 Conn_02x08_Top_Bottom, J2 AudioJack3_Switch

Commit message: OASIS mic updates, audio layout madness
Connections:
- net GND: now also J2.SN; no longer J2.S
Changed lines of the file:
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@@
 	(wire
 		(pts
-			(xy 170.18 78.74) (xy 166.37 78.74)
+			(xy 170.18 81.28) (xy 166.37 81.28)
 		)
 		(stroke
@@
 	(wire
 		(pts
-			(xy 166.37 78.74) (xy 166.37 95.25)
+			(xy 166.37 81.28) (xy 166.37 95.25)
 		)
 		(stroke
