File: PCBs/OASIS_Mic_Card_v1/OASIS_Card.kicad_pcb (KiCad board)
At the start: 2 copper layers, 106.4 x 46.2 mm, 59 parts, among them J1 Conn_02x08_Top_Bottom, J3 AudioJack3_Switch, J5 Control Signals Out, J7 Piggyback Master, J8 Piggyback Slave, J9 12v DC, U1 CD4051B, U3 LTC1044

Commit message: OASIS mic updates, audio layout madness
Parts:
- added C12: 100uF, Capacitor_THT:C_Radial_D6.3mm_H11.0mm_P2.50mm, F.Cu at (122.9, 96.8)
- moved C11 5.62 mm to (115.8, 91.1), turned to -90 degrees
- moved C21 4.53 mm to (180.3, 89.7)
- moved C10 2.07 mm to (118.6, 91.1), turned to -90 degrees
- moved C22 0.70 mm to (175.0, 98.3)
- renumbered C13 to C21, C12 to C22
Routing:
- net +12V: track 213.3 -> 210.6 mm
- net Net-(U3-CAP-): track 3.71 -> 2.95 mm
- net -5V: track 118.5 -> 118.0 mm
- net Net-(U3-CAP+): track 3.46 -> 2.95 mm
- net GND: vias 21 -> 22
Other:
- board text added: "- Update rear silkscreen"
- board text removed: "- Update rear silkscreen - Test LTC1044 circuit - voltage smoothing"
